Commit message: fix(franka-panda-fem-simple-v4-with-arm): replace invalid (+2 more)

File: franka_description/robots/franka_panda_fem_simple_v4_with_arm.urdf (robot description, URDF)
Before this commit: robot panda, 17 links, 16 joints
Links:
- link panda_hand: geometry collision mesh filename=package://franka_description/meshes/collision/hand.obj; visual mesh filename=package://franka_description/meshes/visual/hand.obj
- link panda_left_finger_rigid: geometry collision mesh filename=franka_description/meshes/custom/full_fillet_finger.obj; visual mesh filename=package://franka_description/meshes/custom/full_fillet_fing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
Joints:
- joint rev_jointx: limit lower=-3.14 upper=3.14 effort=1e9.0 velocity=1e9 -> lower=-3.14 upper=3.14 effort=1e9 velocity=1e9
